Commit message: Added world link and base to world joint.

File: scara_description/urdf/scara.xacro (robot description, xacro)
@@ -4,4 +4,6 @@
 <xacro:include filename="$(find scara_description)/urdf/scara.trans" />
 <xacro:include filename="$(find scara_description)/urdf/scara.gazebo" />
+<link name="world">
+</link>
 <link name="base_link">
   <inertial>
@@ -844,4 +846,8 @@
   </collision>
 </link>
+<joint name="world_connect" type="fixed">
+	<parent link="world"/>
+	<child link="base_link"/>
+</joint>
 <joint name="Rigid1" type="fixed">
   <origin rpy="0 0 0" xyz="-0.0211 -0.04 0.05"/>
